File: ground-side-power/GSPD Board.kicad_sch (KiCad schematic)
At the start: 41 parts, among them K1 AZ2150-1A-12DEF, U1 K7805-3AR3, U2 URB2424LD-20WR3

Commit message: Resolved Remaining Schematic Issues
Parts:
- gave numbers to parts that had none: 20
- renumbered C8 to C10, C2 to C7, C6 to C8, C7 to C9, D4 to D5, F3 to F2, F2 to F3, R1 to R2, R2 to R6, R4 to R8
Connections:
- net 12V_Sense-A renamed 12V_Sense+
- net 24V_Sense-A renamed 24V_Sense+
- net 5V_Sense-A renamed 5V_Sense+
- net Sys_Sense-A renamed Sys_Sense+
- no-connect marks 9 -> 10
Other:
- sheet M12 Connections and DAQ Voltage_Current Monitoring ports: added 12V_Sense+, 12V_Sense-, 24V_Sense+, 24V_Sense-, 5V_Sense+, 5V_Sense-, Sys_Sense+, Sys_Sense-; removed 12V_Sense-A, 12V_Sense-B, 24V_Sense-A, 24V_Sense-B, 5V_Sense-A, 5V_Sense-B, Sys_Sense-A, Sys_Sense-B
- moved on the sheet: J1, J2, J3, J4
