File: ground-side-power/GSPD Board.kicad_pcb (KiCad board)
At the start: 2 copper layers, 66 parts, among them J1 Battery Terminals, J10 To DAQ Laptop, J11 To Ethernet, J12 To 5V M12, J13 To DAQ, J14 Extra M12, J15 Extra M12, J16 Extra M12, J17 DAQ Voltage Sensing, J18 DAQ Current Sensing, J2 Battery Terminals, J3 Battery Terminals, J4 Battery Terminals, J5 455860005, J6 455860005, J7 ATX-24, J8 To Router, J9 To RLCS, K1 AZ2150-1A-12DEF, SW1 GRB234A2NABA1, U1 K7805-3AR3, U2 URB2424LD-20WR3, U3 INA180, U4 INA180, U5 INA180, U6 INA180

Commit message: Split into multiple boards
Parts:
- moved J10 577.8 mm to (648.0, 148.2)
- moved J11 556.4 mm to (626.4, 161.9)
- moved J15 556.3 mm to (626.6, 174.9)
- moved J13 553.3 mm to (648.1, 174.8)
- moved J14 553.2 mm to (647.8, 161.9)
- moved J12 535.2 mm to (605.1, 174.8)
- moved J16 507.0 mm to (626.5, 148.3)
- moved J9 486.4 mm to (605.0, 161.9)
- moved J8 485.6 mm to (605.1, 148.3)
- moved U2 382.9 mm to (467.6, 147.0), turned to 90 degrees
- moved SW1 365.3 mm to (422.6, -0.88)
- moved ICL1 361.1 mm to (432.9, 13.3), turned to 180 degrees
- moved J1 360.0 mm to (410.0, -3.63), turned to -90 degrees
- moved J7 348.8 mm to (467.2, 48.9), turned to -90 degrees
- moved J17 331.2 mm to (422.9, 176.9)
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Other:
- board text added: "PSU"

Commit message: Created layout for the footprints for each board
Parts:
- added C15: 100uF, Capacitor_SMD:C_1206_3216Metric_Pad1.33x1.80mm_HandSolder, F.Cu at (105.1, 137.2)
- added C16: 10uF, Capacitor_SMD:C_0603_1608Metric_Pad1.08x0.95mm_HandSolder, F.Cu at (114.0, 137.2)
- added J19: Conn_01x02_Female, GSP:OSTTA020161, F.Cu at (193.0, 78.7)
- added J20: To Ethernet, GSP:EB21A-04-D, F.Cu at (260.9, 146.8)
- added J21: To 5V M12, GSP:EB21A-04-D, F.Cu at (259.1, 120.1)
- added J22: To DAQ, GSP:EB21A-04-D, F.Cu at (207.0, 146.8)
- added J23: Extra M12, GSP:EB21A-04-D, F.Cu at (217.9, 58.9)
- added J24: Extra M12, GSP:EB21A-04-D, F.Cu at (191.2, 58.9)
- added J25: Extra M12, GSP:EB21A-04-D, F.Cu at (244.6, 58.9)
- added J26: Conn_01x02_Female, GSP:OSTTA020161, F.Cu at (109.0, 91.4)
- added J27: Conn_01x02_Female, GSP:OSTTA020161, F.Cu at (103.9, 52.1)
- C10: value 10uF -> 22uF
- C11, C12: value 0.1u -> 10uF; footprint Capacitor_SMD:C_0805_2012Metric_Pad1.18x1.45mm_HandSolder -> Capacitor_SMD:C_0603_1608Metric_Pad1.08x0.95mm_HandSolder
- C14: value 0.1u -> 100uF; footprint Capacitor_SMD:C_0805_2012Metric_Pad1.18x1.45mm_HandSolder -> Capacitor_SMD:C_1206_3216Metric_Pad1.33x1.80mm_HandSolder
- C5: value 22uF -> 22mF; footprint Capacitor_SMD:C_0603_1608Metric_Pad1.08x0.95mm_HandSolder -> GSP:LLS1C223MELZ
- C6: value 10uF -> 22mF; footprint Capacitor_SMD:C_0603_1608Metric_Pad1.08x0.95mm_HandSolder -> GSP:LLS1C223MELZ
- C7: value 10uF -> 0.1u; footprint Capacitor_SMD:C_0603_1608Metric_Pad1.08x0.95mm_HandSolder -> Capacitor_SMD:C_0805_2012Metric_Pad1.18x1.45mm_HandSolder
- C8, C9: value 100uF -> 0.1u; footprint Capacitor_SMD:C_1206_3216Metric_Pad1.33x1.80mm_HandSolder -> Capacitor_SMD:C_0805_2012Metric_Pad1.18x1.45mm_HandSolder
- J10: value To DAQ Laptop -> Conn_01x03_Female; footprint GSP:EB21A-04-D -> GSP:TB005-762-03BE
- J11: value To Ethernet -> Conn_01x03_Female; footprint GSP:EB21A-04-D -> GSP:TB005-762-03BE
- J12: value To 5V M12 -> Conn_01x04_Female
- J13: value To DAQ -> DAQ Voltage Sensing
- J14: value Extra M12 -> DAQ Current Sensing
- J15: value Extra M12 -> To Router
- J16: value Extra M12 -> To RLCS
- J17: value DAQ Voltage Sensing -> To DAQ Laptop
- J18: value DAQ Current Sensing -> Conn_01x02_Female; footprint GSP:EB21A-04-D -> GSP:OSTTA020161
- J8: value To Router -> Conn_01x03_Female; footprint GSP:EB21A-04-D -> GSP:TB005-762-03BE
- J9: value To RLCS -> Conn_01x03_Female; footprint GSP:EB21A-04-D -> GSP:TB005-762-03BE
- R12: value 100K -> R_Small_US; footprint Resistor_SMD:R_0402_1005Metric_Pad0.72x0.64mm_HandSolder -> Resistor_SMD:R_1206_3216Metric_Pad1.30x1.75mm_HandSolder
- R3: value 0.0016 -> 220K; footprint Resistor_SMD:R_1206_3216Metric_Pad1.30x1.75mm_HandSolder -> Resistor_SMD:R_0402_1005Metric_Pad0.72x0.64mm_HandSolder
- R4: value 0.01 -> 0.0016
- R5: value R_Small_US -> 100K; footprint Resistor_SMD:R_1206_3216Metric_Pad1.30x1.75mm_HandSolder -> Resistor_SMD:R_0402_1005Metric_Pad0.72x0.64mm_HandSolder
- R7: value 0.04 -> 0.01
- R9: value 220K -> 0.04; footprint Resistor_SMD:R_0402_1005Metric_Pad0.72x0.64mm_HandSolder -> Resistor_SMD:R_1206_3216Metric_Pad1.30x1.75mm_HandSolder
- U1: value K7805-3AR3 -> INA180; footprint GSP:K7805-3AR3 -> Package_TO_SOT_SMD:SOT-23-5_HandSoldering
- U2: value URB2424LD-20WR3 -> INA180; footprint GSP:URB2424LD-20WR3 -> Package_TO_SOT_SMD:SOT-23-5_HandSoldering
- U3: value INA180 -> K7805-3AR3; footprint Package_TO_SOT_SMD:SOT-23-5_HandSoldering -> GSP:K7805-3AR3
- U6: value INA180 -> URB2424LD-20WR3; footprint Package_TO_SOT_SMD:SOT-23-5_HandSoldering -> GSP:URB2424LD-20WR3
- moved J10 600.1 mm to (50.7, 90.3)
- moved J11 551.2 mm to (79.9, 90.3)
- moved J8 549.1 mm to (64.5, 52.1), turned to 180 degrees
- moved J9 524.3 mm to (92.3, 51.9), turned to 180 degrees
- moved J13 509.7 mm to (139.4, 143.5), turned to 180 degrees
- moved J14 505.4 mm to (143.2, 132.1), turned to 90 degrees
- moved J12 467.1 mm to (143.2, 105.4), turned to 90 degrees
- moved U2 415.6 mm to (98.8, -44.5), turned to 180 degrees
- moved U1 399.0 mm to (50.5, 8.89)
- moved C2 382.2 mm to (69.6, -37.4), turned to -90 degrees
- moved J15 382.1 mm to (259.3, 69.3), turned to -90 degrees
- moved SW1 379.7 mm to (49.3, -70.0), turned to 90 degrees
- moved J4 374.9 mm to (49.3, -58.6)
- moved J16 371.3 mm to (259.1, 94.7), turned to -90 degrees
- moved J2 365.7 mm to (49.3, -28.1)
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Connections:
- net /ACPowerSupply renamed /Input/ACPowerSupply
- net /BatteryPowerSupply renamed /Input/BatteryPowerSupply
- C10 pad 1: +24V -> Net-(C10-Pad1)
- C11 pad 1: GND -> +BATT
- C11 pad 2: +5V -> GND
- C12 pad 1: GND -> +5V
- C12 pad 2: +5V -> GND
- C14 pad 1: GND -> +BATT
- C14 pad 2: +5V -> GND
- C5 pad 1: Net-(C5-Pad1) -> +12V
- C6 pad 1: +BATT -> +12V
- C7 pad 1: +5V -> GND
- C7 pad 2: GND -> +5V
- C8 pad 1: +BATT -> GND
- C8 pad 2: GND -> +5V
- C9 pad 1: Net-(C9-Pad1) -> GND
- C9 pad 2: GND -> +5V
- F2 pad 2: /12V_Sense+ -> /Input/12V_Sense+
- F3 pad 1: Net-(C5-Pad1) -> Net-(C10-Pad1)
- F3 pad 2: /5V_Sense+ -> /Converters/5V_Sense+
- F4 pad 1: Net-(C9-Pad1) -> Net-(C15-Pad1)
- F4 pad 2: /24V_Sense+ -> /Converters/24V_Sense+
- J10 pad 1: +24V -> +BATT
- J10 pad 3: +5V -> GND
- J11 pad 1: +24V -> /Converters/12V_OUT
- J11 pad 2: +12V -> /Converters/TOTAL_OUT
- J11 pad 3: +5V -> /Converters/12_VOLTAGE
- J12 pad 1: +24V -> +5V
- J12 pad 3: +5V -> +24V
- J13 pad 1: +24V -> +BATT
- J13 pad 2: +12V -> /Converters/5V_VOLTAGE
- J13 pad 3: +5V -> /Converters/12_VOLTAGE
- J13 pad 4: GND -> /Converters/24V_VOLTAGE
- J14 pad 1: +24V -> /Converters/TOTAL_OUT
- J14 pad 2: +12V -> /Converters/5V_OUT
- J14 pad 3: +5V -> /Converters/12V_OUT
- J14 pad 4: GND -> /Converters/24V_OUT
- J17 pad 1: +BATT -> +24V
- J17 pad 2: /M12 Connections and DAQ Voltage_Current Monitoring/5V_VOLTAGE -> +12V
- J17 pad 3: /M12 Connections and DAQ Voltage_Current Monitoring/12V_VOLTAGE -> +5V
- J17 pad 4: /M12 Connections and DAQ Voltage_Current Monitoring/24V_VOLTAGE -> GND
- J18 pad 1: /M12 Connections and DAQ Voltage_Current Monitoring/TOTAL_OUT -> +12V
- J18 pad 2: /M12 Connections and DAQ Voltage_Current Monitoring/5V_OUT -> +24V
- J8 pad 1: +24V -> +12V
- J8 pad 2: +12V -> +BATT
- J8 pad 3: +5V -> GND
- J9 pad 1: +24V -> /Converters/12V_OUT
- J9 pad 2: +12V -> /Converters/TOTAL_OUT
- J9 pad 3: +5V -> /Converters/12_VOLTAGE
- K1 pad 2: /Sys_Sense+ -> /Input/Sys_Sense+
- R1 pad 1: /Sys_Sense+ -> /Input/Sys_Sense+
- R10 pad 2: /M12 Connections and DAQ Voltage_Current Monitoring/24V_VOLTAGE -> /Converters/24V_VOLTAGE
- R11 pad 2: /M12 Connections and DAQ Voltage_Current Monitoring/5V_VOLTAGE -> /Converters/5V_VOLTAGE
- R12 pad 1: /M12 Connections and DAQ Voltage_Current Monitoring/12V_VOLTAGE -> GND
- R12 pad 2: GND -> Net-(D6-Pad1)
- R13 pad 1: /M12 Connections and DAQ Voltage_Current Monitoring/24V_VOLTAGE -> /Converters/24V_VOLTAGE
- R14 pad 1: /M12 Connections and DAQ Voltage_Current Monitoring/5V_VOLTAGE -> /Converters/5V_VOLTAGE
- R3 pad 1: /12V_Sense+ -> +12V
- R3 pad 2: +12V -> /Converters/12_VOLTAGE
- R4 pad 1: /5V_Sense+ -> /Input/12V_Sense+
- R4 pad 2: +5V -> +12V
- R5 pad 1: GND -> /Converters/12_VOLTAGE
- R5 pad 2: Net-(D4-Pad1) -> GND
- R6 pad 2: Net-(D5-Pad1) -> Net-(D4-Pad1)
- R7 pad 1: +24V -> /Converters/5V_Sense+
- R7 pad 2: /24V_Sense+ -> +5V
- R8 pad 2: Net-(D6-Pad1) -> Net-(D5-Pad1)
- R9 pad 1: +12V -> +24V
- R9 pad 2: /M12 Connections and DAQ Voltage_Current Monitoring/12V_VOLTAGE -> /Converters/24V_Sense+
- U1 pad 1: unconnected-(U1-Pad1) -> /Converters/12V_OUT
- U1 pad 2: +BATT -> GND
- U1 pad 3: +BATT -> /Input/12V_Sense+
- U1 pad 4: +BATT -> +12V
- U1 pad 5: GND -> +5V
- U2 pad 1: unconnected-(U2-Pad1) -> /Converters/TOTAL_OUT
- U2 pad 3: +BATT -> /Input/Sys_Sense+
- U2 pad 4: Net-(C9-Pad1) -> +BATT
- U2 pad 5: GND -> +5V
- U3 pad 1: /M12 Connections and DAQ Voltage_Current Monitoring/TOTAL_OUT -> unconnected-(U3-Pad1)
- U3 pad 2: GND -> +BATT
- U3 pad 3: /Sys_Sense+ -> +BATT
- U3 pad 5: +5V -> GND
- U4 pad 1: /M12 Connections and DAQ Voltage_Current Monitoring/5V_OUT -> /Converters/5V_OUT
- U4 pad 3: /5V_Sense+ -> /Converters/5V_Sense+
- U5 pad 1: /M12 Connections and DAQ Voltage_Current Monitoring/12V_OUT -> /Converters/24V_OUT
- U5 pad 3: /12V_Sense+ -> /Converters/24V_Sense+
- U5 pad 4: +12V -> +24V
- U6 pad 1: /M12 Connections and DAQ Voltage_Current Monitoring/24V_OUT -> unconnected-(U6-Pad1)
- U6 pad 3: /24V_Sense+ -> +BATT
- U6 pad 4: +24V -> Net-(C15-Pad1)
- U6 pad 5: +5V -> GND
Other:
- board text removed: "PSU"

Commit message: Added Fan Headers + Thermistor
Parts:
- added M1: Fan_PC_Chassis, Connector:FanPinHeader_1x03_P2.54mm_Vertical, F.Cu at (9.65, -260.2)
- added M2: Fan_PC_Chassis, Connector:FanPinHeader_1x03_P2.54mm_Vertical, F.Cu at (294.2, -88.5)
- added R15: B57621C5103K062, Resistor_SMD:R_1206_3216Metric_Pad1.30x1.75mm_HandSolder, F.Cu at (74.1, -40.8)
- added R16: 10K, Resistor_SMD:R_0402_1005Metric_Pad0.72x0.64mm_HandSolder, F.Cu at (72.7, -38.2)
- moved J26 220.4 mm to (47.5, -120.3)
- moved C10 183.4 mm to (28.9, -61.2)
- moved C11 183.4 mm to (56.8, -43.5)
- moved C12 183.4 mm to (37.8, -61.2)
- moved C13 183.4 mm to (68.3, -65.0)
- moved C8 183.4 mm to (-6.42, -159.0)
- moved C9 183.4 mm to (59.4, -65.0)
- moved D2 183.4 mm to (67.5, -243.9)
- moved D5 183.4 mm to (45.4, -67.6)
- moved F1 183.4 mm to (67.5, -253.0)
- moved F3 183.4 mm to (28.9, -67.6)
- moved F4 183.4 mm to (48.0, -43.5)
- moved ICL1 183.4 mm to (76.4, -246.7)
- moved J14 183.4 mm to (86.1, -42.2)
- moved J3 183.4 mm to (-7.92, -187.1)
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Connections:
- J13 pad 1: +BATT -> /Converters/Temp
Other:
- board text added: "NOTE: Above boards are to scale and with connect nets, however, changes should be made to induvidual boards in their induvidual files. Update this file by copy pasting boards from the other files. Do NOT use this file for gerbers."

Commit message: Resolved Final Issues
Parts:
- removed C5, C6: 22mF, GSP:LLS1C223MELZ
- removed J11: Conn_01x03_Female, GSP:TB005-762-03BE
- added ?: , clipboard:6b5716c7-8553-4764-af17-05841c85de2e, F.Cu at (30.2, -50.0)
- added ?: , , F.Cu at (18.3, -128.1)
- added ?: , , F.Cu at (293.3, -33.0)
- added ?: , , F.Cu at (111.3, -128.1)
- added ?: , , F.Cu at (205.0, -33.0)
- added ?: , , F.Cu at (293.3, -92.6)
- added ?: , clipboard:6b5716c7-8553-4764-af17-05841c85de2e, F.Cu at (102.9, -114.6)
- added ?: , , F.Cu at (111.3, -239.5)
- added ?: , clipboard:6b5716c7-8553-4764-af17-05841c85de2e, F.Cu at (30.2, -114.6)
- added ?: , clipboard:6b5716c7-8553-4764-af17-05841c85de2e, F.Cu at (102.9, -50.1)
- added ?: , clipboard:ee0da358-bf61-46f9-af96-80582bde7c0f, F.Cu at (18.3, -239.5)
- added G***: LOGO, rlcs:rocketry_logo_small, F.Cu at (35.4, -235.8)
- added G***: LOGO, rlcs:rocketry_logo_small, F.Cu at (216.1, -90.5)
- added G***: LOGO, rlcs:rocketry_logo_small, F.Cu at (65.3, -105.9)
- added R17: 10k, Resistor_SMD:R_0805_2012Metric_Pad1.20x1.40mm_HandSolder, F.Cu at (81.0, -223.9)
- added REF**: MountingHole_3.2mm_M3_Pad, MountingHole:MountingHole_3.2mm_M3_Pad, F.Cu at (205.0, -92.6)
- C1, C14, C15: footprint Capacitor_SMD:C_1206_3216Metric_Pad1.33x1.80mm_HandSolder -> Capacitor_THT:CP_Radial_D6.3mm_P2.50mm
- C10, C11: footprint Capacitor_SMD:C_0603_1608Metric_Pad1.08x0.95mm_HandSolder -> Capacitor_SMD:C_0805_2012Metric_Pad1.18x1.45mm_HandSolder; moved to B.Cu
- C12, C16: footprint Capacitor_SMD:C_0603_1608Metric_Pad1.08x0.95mm_HandSolder -> Capacitor_SMD:C_0805_2012Metric_Pad1.18x1.45mm_HandSolder
- C13, C7, C8, C9, R15, U1, U2, U4, U5: moved to B.Cu
- D1: footprint Capacitor_SMD:C_0603_1608Metric_Pad1.08x0.95mm_HandSolder -> Diode_SMD:D_SMB_Handsoldering; moved to B.Cu
- D2: footprint Diode_SMD:D_SMB -> Diode_SMD:D_SMB_Handsoldering; moved to B.Cu
- D3, D4, D5, D6: footprint Diode_SMD:D_0805_2012Metric -> Diode_SMD:D_1206_3216Metric_Pad1.42x1.75mm_HandSolder
- F1, F2, F3, F4: footprint Fuse:Fuse_1206_3216Metric_Pad1.42x1.75mm_HandSolder -> Fuse:Fuseholder_Clip-6.3x32mm_Littelfuse_102_122_Inline_P34.21x7.62mm_D1.98mm_Horizontal
- J1, J18, J2, J26, J27, J3, J4: footprint GSP:OSTTA020161 -> GSP:1935310
- J10: footprint GSP:TB005-762-03BE -> GSP:1935310
- J12, J13: footprint GSP:EB21A-04-D -> GSP:1935323
- J14: footprint GSP:EB21A-04-D -> GSP:1935310
- J15, J16, J17, J20, J21, J22, J23, J24, J25: footprint GSP:EB21A-04-D -> GSP:CUI_TB008A-508-04BE
- J19: footprint GSP:OSTTA020161 -> GSP:1935323
- J5, J6: value 455860005 -> 874270842; footprint GSP:MOLEX_455860005 -> GSP:MOLEX_874270842
- J7: footprint GSP:MOLEX_15246240 -> GSP:MOLEX_442060001
- J8, J9, SW1: footprint GSP:TB005-762-03BE -> GSP:1935323
- R1, R4: value 0.0016 -> 0.0015; footprint Resistor_SMD:R_1206_3216Metric_Pad1.30x1.75mm_HandSolder -> Resistor_SMD:R_2512_6332Metric_Pad1.40x3.35mm_HandSolder; moved to B.Cu
- R10, R11: footprint Resistor_SMD:R_0603_1608Metric_Pad0.98x0.95mm_HandSolder -> Resistor_SMD:R_0805_2012Metric_Pad1.20x1.40mm_HandSolder; moved to B.Cu
- R12, R2, R6, R8: footprint Resistor_SMD:R_1206_3216Metric_Pad1.30x1.75mm_HandSolder -> Resistor_SMD:R_0805_2012Metric_Pad1.20x1.40mm_HandSolder
- R13, R14, R16: footprint Resistor_SMD:R_0402_1005Metric_Pad0.72x0.64mm_HandSolder -> Resistor_SMD:R_0805_2012Metric_Pad1.20x1.40mm_HandSolder; moved to B.Cu
- R3, R5: footprint Resistor_SMD:R_0402_1005Metric_Pad0.72x0.64mm_HandSolder -> Resistor_SMD:R_0805_2012Metric_Pad1.20x1.40mm_HandSolder
- R7, R9: footprint Resistor_SMD:R_1206_3216Metric_Pad1.30x1.75mm_HandSolder -> Resistor_SMD:R_2512_6332Metric_Pad1.40x3.35mm_HandSolder; moved to B.Cu
- moved MES1 107.2 mm to (23.9, -152.5), turned to -90 degrees
- moved M2 97.1 mm to (214.1, -33.7), turned to 0 degrees
- moved M1 97.0 mm to (23.8, -164.2), turned to -90 degrees
- moved C2 80.2 mm to (75.2, -161.7), turned to 0 degrees
- moved R2 80.0 mm to (20.3, -140.3), turned to 0 degrees
- moved J20 73.7 mm to (252.5, -92.6), turned to -90 degrees
- moved C3 72.9 mm to (75.7, -209.7), turned to 0 degrees
- moved R4 70.4 mm to (63.5, -166.7), turned to -90 degrees
- moved C4 70.0 mm to (75.4, -185.5), turned to 0 degrees
- moved SW1 70.0 mm to (61.3, -234.0), turned to 0 degrees
- moved D3 69.7 mm to (25.7, -140.3), turned to 0 degrees
- moved D4 65.4 mm to (60.5, -154.3), turned to 90 degrees
- moved R12 64.2 mm to (104.9, -60.3), turned to 180 degrees
- moved C12 63.6 mm to (98.3, -81.0)
- moved R6 63.4 mm to (60.5, -147.7), turned to 90 degrees
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Connections:
- F2 pad 2: /Input/12V_Sense+ -> (no net)
- F3 pad 2: /Converters/5V_Sense+ -> (no net)
- F4 pad 2: /Converters/24V_Sense+ -> (no net)
- J1 pad 1: /Input/BatteryPowerSupply -> (no net)
- J10 pad 1: +BATT -> GND
- J10 pad 2: +12V -> +BATT
- J12 pad 1: +5V -> +24V
- J12 pad 2: +12V -> GND
- J12 pad 3: +24V -> +5V
- J13 pad 1: /Converters/Temp -> (no net)
- J13 pad 2: /Converters/5V_VOLTAGE -> (no net)
- J13 pad 3: /Converters/12_VOLTAGE -> (no net)
- J14 pad 1: /Converters/TOTAL_OUT -> (no net)
- J14 pad 2: /Converters/5V_OUT -> (no net)
- J18 pad 2: +24V -> GND
- J19 pad 1: +5V -> +24V
- J2 pad 1: /Input/BatteryPowerSupply -> (no net)
- J27 pad 1: +5V -> GND
- J27 pad 2: GND -> +5V
- J3 pad 1: /Input/BatteryPowerSupply -> (no net)
- J4 pad 1: /Input/BatteryPowerSupply -> (no net)
- J5 pad 1: /Input/ACPowerSupply -> (no net)
- J5 pad 2: /Input/ACPowerSupply -> (no net)
- J5 pad 3: /Input/ACPowerSupply -> (no net)
- J6 pad 1: /Input/ACPowerSupply -> (no net)
- J6 pad 2: /Input/ACPowerSupply -> (no net)
- J6 pad 3: /Input/ACPowerSupply -> (no net)
- J7 pad 10: /Input/ACPowerSupply -> (no net)
- J7 pad 11: /Input/ACPowerSupply -> (no net)
- J9 pad 1: /Converters/12V_OUT -> (no net)
- J9 pad 2: /Converters/TOTAL_OUT -> (no net)
- J9 pad 3: /Converters/12_VOLTAGE -> (no net)
- K1 pad 2: /Input/Sys_Sense+ -> (no net)
- R1 pad 1: /Input/Sys_Sense+ -> (no net)
- R10 pad 2: /Converters/24V_VOLTAGE -> (no net)
- R11 pad 2: /Converters/5V_VOLTAGE -> (no net)
- R13 pad 1: /Converters/24V_VOLTAGE -> (no net)
- R14 pad 1: /Converters/5V_VOLTAGE -> (no net)
- R15 pad 2: /Converters/Temp -> (no net)
- R16 pad 1: /Converters/Temp -> (no net)
- R3 pad 2: /Converters/12_VOLTAGE -> (no net)
- R4 pad 1: /Input/12V_Sense+ -> (no net)
- R5 pad 1: /Converters/12_VOLTAGE -> (no net)
- R7 pad 1: /Converters/5V_Sense+ -> (no net)
- R9 pad 2: /Converters/24V_Sense+ -> (no net)
- SW1 pad 1: /Input/ACPowerSupply -> (no net)
- SW1 pad 3: /Input/BatteryPowerSupply -> (no net)
- U1 pad 1: /Converters/12V_OUT -> (no net)
- U1 pad 3: /Input/12V_Sense+ -> (no net)
- U2 pad 1: /Converters/TOTAL_OUT -> (no net)
- U2 pad 3: /Input/Sys_Sense+ -> (no net)
- U4 pad 1: /Converters/5V_OUT -> (no net)
- U4 pad 3: /Converters/5V_Sense+ -> (no net)
- U5 pad 1: /Converters/24V_OUT -> (no net)
- U5 pad 3: /Converters/24V_Sense+ -> (no net)
Routing:
- net (no net): track 0.00 -> 376.9 mm, vias 0 -> 4
- net +12V: track 0.00 -> 318.6 mm
- net +5V: track 0.00 -> 317.6 mm, vias 0 -> 5
- net GND: track 0.00 -> 291.7 mm, vias 0 -> 7
- net +24V: track 0.00 -> 92.7 mm, vias 0 -> 1
- net Net-(C10-Pad1): track 0.00 -> 29.3 mm
- net +BATT: track 0.00 -> 17.6 mm
- net Net-(D4-Pad1): track 0.00 -> 4.12 mm
- net Net-(D6-Pad1): track 0.00 -> 3.61 mm
- net Net-(D3-Pad1): track 0.00 -> 2.85 mm
- net Net-(D5-Pad1): track 0.00 -> 2.59 mm
- added copper zone on B.Cu, net (none)
- added copper zone on B.Cu, net +12V
- added copper zone on B.Cu, net +24V
- added copper zone on F.Cu, net +24V
- added copper zone on B.Cu, net +5V
- added copper zone on B.Cu, net +BATT
- added copper zone on F.Cu, net GND
- added copper zone on B.Cu, net Net-(C15-Pad1)
- added copper zone on B.Cu, net Net-(D1-Pad1)
- added copper zone on B.Cu, net Net-(D2-Pad2)
- added copper zone on B.Cu, net Net-(F1-Pad1)
- added copper zone on B.Cu, net Net-(F1-Pad2)
Other:
- board outline added: 284.1 x 215.3 mm
- board text added: "+"
- board text added: "+12"
- board text added: "+12 Current"
- board text added: "+12 Voltage"
- board text added: "+24"
- board text added: "+5"
- board text added: "+BATT"
- board text added: "-"
- board text added: "0"
- board text added: "AC"
- board text added: "DC"
- board text added: "Don't Populate"
- board text added: "Ground Side Power Connector Board Domenic Hampson Elias Kountouris"
- board text added: "Ground Side Power Converter Board Domenic Hampson Elias Kountouris"
- board text added: "Ground Side Power Input Board Domenic Hampson Elias Kountouris"
- board text added: "SWITCH"
- board text added: "Temp"
- board text added: "Total Current"

Commit message: Silkscreen and current sense changes
Parts:
- removed the ? at (30.2, -50.0)
- removed the ? at (18.3, -128.1)
- removed the ? at (293.3, -33.0)
- removed the ? at (111.3, -128.1)
- removed the ? at (205.0, -33.0)
- removed the ? at (293.3, -92.6)
- removed the ? at (102.9, -114.6)
- removed the ? at (111.3, -239.5)
- removed the ? at (30.2, -114.6)
- removed the ? at (102.9, -50.1)
- removed the G*** at (35.4, -235.8)
- removed the G*** at (216.1, -90.5)
- removed the G*** at (65.3, -105.9)
- added ?: , , F.Cu at (298.4, -34.3)
- added ?: , clipboard:6b5716c7-8553-4764-af17-05841c85de2e, F.Cu at (28.1, -113.9)
- added ?: , clipboard:6b5716c7-8553-4764-af17-05841c85de2e, F.Cu at (100.7, -49.5)
- added ?: , , F.Cu at (210.1, -34.3)
- added ?: , , F.Cu at (298.4, -93.9)
- added ?: , , F.Cu at (107.6, -131.3)
- added ?: , clipboard:6b5716c7-8553-4764-af17-05841c85de2e, F.Cu at (100.7, -113.9)
- added ?: , , F.Cu at (21.0, -131.2)
- added ?: , , F.Cu at (107.6, -244.6)
- added ?: , clipboard:6b5716c7-8553-4764-af17-05841c85de2e, F.Cu at (28.1, -49.4)
- added G***: LOGO, rlcs:rocketry_logo_small, F.Cu at (38.1, -240.9)
- added G***: LOGO, rlcs:rocketry_logo_small, F.Cu at (63.2, -105.3)
- added G***: LOGO, rlcs:rocketry_logo_small, F.Cu at (221.0, -90.4)
- J8: footprint GSP:1935323 -> GSP:CUI_TB008A-508-04BE
- moved C2 49.6 mm to (79.1, -211.1)
- moved C4 27.5 mm to (79.1, -158.3)
- moved C3 25.2 mm to (79.1, -184.7)
- moved M2 20.3 mm to (220.0, -53.1), turned to -90 degrees
- moved D4 14.6 mm to (46.1, -151.8)
- moved R3 14.6 mm to (40.0, -152.3)
- moved R5 14.6 mm to (40.0, -145.2)
- moved R6 14.6 mm to (46.1, -145.2)
- moved J8 7.89 mm to (70.5, -138.4)
- moved U2 6.16 mm to (36.4, -188.0)
- moved ICL1 5.77 mm to (49.7, -219.4)
- moved ? 5.77 mm to (21.0, -244.6)
- moved D2 5.77 mm to (46.4, -212.3)
- moved D1 5.77 mm to (36.7, -203.4)
- moved F2 5.77 mm to (35.6, -178.7)
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Connections:
- J8 pad 2: +BATT -> GND
- J8 pad 3: GND -> +BATT
Routing:
- net +12V: track 318.6 -> 341.1 mm
- net (no net): track 376.9 -> 362.8 mm
- net +5V: track 317.6 -> 331.4 mm
- net GND: track 291.7 -> 289.7 mm
- net +BATT: track 17.6 -> 16.8 mm
Other:
- board size 284.1 x 215.3 mm -> 286.6 x 219.2 mm
- board text added: "+Batt"
- board text added: "Ground Side Power Connector Board Jan 2023 Domenic Hampson Elias Kountouris"
- board text added: "Ground Side Power Converter Board Jan 2023 Domenic Hampson Elias Kountouris"
- board text added: "Ground Side Power Input Board Jan 2023 Domenic Hampson Elias Kountouris"
- board text removed: "Ground Side Power Connector Board Domenic Hampson Elias Kountouris"
- board text removed: "Ground Side Power Converter Board Domenic Hampson Elias Kountouris"
- board text removed: "Ground Side Power Input Board Domenic Hampson Elias Kountouris"

Commit message: Added Gerbers
Parts:
- removed the ? at (28.1, -113.9)
- removed the ? at (100.7, -49.5)
- removed the ? at (107.6, -131.3)
- removed the ? at (100.7, -113.9)
- removed the ? at (21.0, -131.2)
- removed the ? at (107.6, -244.6)
- removed the ? at (28.1, -49.4)
- removed the G*** at (38.1, -240.9)
- removed the G*** at (63.2, -105.3)
- added ?: , clipboard:6b5716c7-8553-4764-af17-05841c85de2e, F.Cu at (30.0, -105.9)
- added ?: , clipboard:6b5716c7-8553-4764-af17-05841c85de2e, F.Cu at (30.0, -41.4)
- added ?: , , F.Cu at (18.5, -128.2)
- added ?: , clipboard:6b5716c7-8553-4764-af17-05841c85de2e, F.Cu at (102.6, -105.9)
- added ?: , , F.Cu at (105.1, -241.6)
- added ?: , , F.Cu at (105.1, -128.2)
- added ?: , clipboard:6b5716c7-8553-4764-af17-05841c85de2e, F.Cu at (102.6, -41.5)
- added G***: LOGO, rlcs:rocketry_logo_small, F.Cu at (35.6, -237.9)
- added G***: LOGO, rlcs:rocketry_logo_small, F.Cu at (65.1, -97.3)
- MES1: footprint GSP:OSTTA020161 -> GSP:1935310
- moved C11 8.22 mm to (40.4, -81.7)
- moved C12 8.22 mm to (98.0, -72.4)
- moved C15 8.22 mm to (71.1, -38.5)
- moved C16 8.22 mm to (97.9, -54.3)
- moved C9 8.22 mm to (82.7, -76.3)
- moved D5 8.22 mm to (98.6, -75.1)
- moved F3 8.22 mm to (65.0, -82.4)
- moved J10 8.22 mm to (49.8, -96.3)
- moved J27 8.22 mm to (86.4, -96.3)
- moved R10 8.22 mm to (41.9, -35.7)
- moved R11 8.22 mm to (52.1, -35.7)
- moved R13 8.22 mm to (37.3, -35.7)
- moved R15 8.22 mm to (62.5, -35.7)
- moved R16 8.22 mm to (57.1, -35.7)
- moved R8 8.22 mm to (103.6, -75.1)
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Routing:
- net +BATT: track 16.8 -> 23.3 mm
Other:
- board size 286.6 x 219.2 mm -> 289.1 x 216.1 mm
