File: ground-side-power/Converters/Converters.kicad_sch (KiCad schematic)
At the start: 46 parts, among them J1 DAQ Voltage Sensing, J2 DAQ Current Sensing, J3 Ground Connections, J4 BATT_IN, J5 POWER_OUT, J6 5V_IN, U1 K7805-3AR3, U2 TPS55340, U3 INA180, U4 INA180

Commit message: added inductor footprint
Parts:
- L1: footprint Inductor_SMD:L_0805_2012Metric_Pad1.15x1.40mm_HandSolder -> ETQ-P5M100YFC:ETQP5M_YFC_YGC
Connections:
- net 24V_OUT: now also J2.2 (Pin_2); no longer J2.1 (Pin_1)
- net 5V_OUT: now also J2.1 (Pin_1); no longer J2.2 (Pin_2)
Changed lines of the file:
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@@
     (effects (font (size 1.27 1.27)) (justify right bottom))
   )
-  (label "24V_OUT" (at 96.52 172.72 180) (fields_autoplaced)
+  (label "24V_OUT" (at 96.52 175.26 180) (fields_autoplaced)
     (effects (font (size 1.27 1.27)) (justify right bottom))
   )
@@
     (effects (font (size 1.27 1.27)) (justify right bottom))
   )
-  (label "5V_OUT" (at 96.52 175.26 180) (fields_autoplaced)
+  (label "5V_OUT" (at 96.52 172.72 180) (fields_autoplaced)
     (effects (font (size 1.27 1.27)) (justify right bottom))
   )
@@
       (effects (font (size 1.27 1.27)))
     )
-    (property "Footprint" "Inductor_SMD:L_0805_2012Metric_Pad1.15x1.40mm_HandSolder" (at 33.02 40.64 0)
+    (property "Footprint" "ETQ-P5M100YFC:ETQP5M_YFC_YGC" (at 33.02 40.64 0)
       (effects (font (size 1.27 1.27)) hide)
     )
@@
       (effects (font (size 1.27 1.27)) hide)
     )
-    (property "Datasheet" "" (at 53.34 67.31 0)
-      (effects (font (size 1.27 1.27)) hide)
-    )
+    (property "Datasheet" "https://www.ti.com/lit/ds/symlink/tps55340.pdf?HQS=dis-dk-null-digikeymode-dsf-pf-null-wwe&ts=1709403385904&ref_url=https%253A%252F%252Fwww.ti.com%252Fgeneral%252Fdocs%252Fsuppproductinfo.tsp%253FdistId%253D10%2526gotoUrl%253Dhttps%253A%252F%252Fwww.ti.com%252Flit%252Fgpn%252Ftps55340" (at 53.34 67.31 0)
+      (effects (font (size 1.27 1.27)) hide)
+    )
