File: ground-side-power/Converters/Converters.kicad_pcb (KiCad board)
At the start: 2 copper layers, 82.8 x 74.4 mm, 51 parts, among them J1 DAQ Voltage Sensing, J2 DAQ Current Sensing, J3 Ground Connections, J4 BATT_IN, J5 POWER_OUT, J6 5V_IN, U1 K7805-3AR3, U2 TPS55340, U3 INA180, U4 INA180

Commit message: implemented comments
Parts:
- moved +BATT 0.55 mm to (181.3, 125.8)
Routing:
- net +24V: track 97.2 -> 98.1 mm
Changed lines of the file:
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@@
   )
   (footprint "TestPoint:TestPoint_Plated_Hole_D2.0mm" (layer "F.Cu")
-    (at 181.7 126.1 90)
+    (at 181.2544 125.7808 90)
     (descr "Plated Hole as test Point, diameter 2.0mm")
     (tags "test point plated hole")
@@
   (segment (start 152.24 123.129923) (end 154.686 123.129923) (width 0.25) (layer "F.Cu") (net 2))
   (segment (start 164.766 122.447923) (end 166.116 122.447923) (width 0.25) (layer "F.Cu") (net 2))
-  (segment (start 148.844 121.765923) (end 149.86 120.749923) (width 0.25) (layer "F.Cu") (net 2))
   (segment (start 168.154077 101.445923) (end 175 94.6) (width 0.25) (layer "F.Cu") (net 2))
   (segment (start 164.338 122.019923) (end 164.766 122.447923) (width 0.25) (layer "F.Cu") (net 2))
@@
   (segment (start 155.702 103.985923) (end 158.242 101.445923) (width 0.25) (layer "F.Cu") (net 2))
   (segment (start 160.274 119.733923) (end 160.274 117.701923) (width 0.25) (layer "F.Cu") (net 2))
+  (segment (start 148.844 122.682) (end 149.86 121.666) (width 0.25) (layer "F.Cu") (net 2))
   (segment (start 154.686 123.129923) (end 158.374 123.129923) (width 0.25) (layer "F.Cu") (net 2))
   (segment (start 155.702 113.129923) (end 155.702 103.985923) (width 0.25) (layer "F.Cu") (net 2))
@@
   (segment (start 167.426 78.545923) (end 159.766 86.205923) (width 0.25) (layer "F.Cu") (net 2))
   (segment (start 164.338 117.955923) (end 164.338 122.019923) (width 0.25) (layer "F.Cu") (net 2))
+  (segment (start 148.844 124.559923) (end 148.844 122.682) (width 0.25) (layer "F.Cu") (net 2))
   (segment (start 172.8 94.6) (end 174 94.6) (width 1.3462) (layer "F.Cu") (net 2))
   (segment (start 166.116 122.447923) (end 168.976 122.447923) (width 0.25) (layer "F.Cu") (net 2))
   (segment (start 177.050077 94.6) (end 178.562 96.111923) (width 1.3462) (layer "F.Cu") (net 2))
+  (segment (start 149.86 121.666) (end 149.86 120.749923) (width 0.25) (layer "F.Cu") (net 2))
   (segment (start 160.274 117.701923) (end 155.702 113.129923) (width 0.25) (layer "F.Cu") (net 2))
   (segment (start 166.878 120.263423) (end 166.878 121.685923) (width 0.25) (layer "F.Cu") (net 2))
@@
   (segment (start 174 94.6) (end 175 94.6) (width 1.3462) (layer "F.Cu") (net 2))
   (segment (start 175.6 93) (end 174 94.6) (width 0.25) (layer "F.Cu") (net 2))
-  (segment (start 148.844 124.559923) (end 148.844 121.765923) (width 0.25) (layer "F.Cu") (net 2))
   (segment (start 175 94.6) (end 176.1 94.6) (width 1.3462) (layer "F.Cu") (net 2))
   (segment (start 176.1 94.6) (end 177.050077 94.6) (width 1.3462) (layer "F.Cu") (net 2))
@@
   (segment (start 170.876 121.831923) (end 171.958 120.749923) (width 0.25) (layer "F.Cu") (net 4))
   (segment (start 175.452039 108.747961) (end 174.5 107.795923) (width 0.25) (layer "F.Cu") (net 4))
-  (segment (start 132.5 136.2) (end 135.845923 139.545923) (width 0.25) (layer "F.Cu") (net 4))
+  (segment (start 173.482 138.021923) (end 173.482 121.3612) (width 0.25) (layer "F.Cu") (net 4))
+  (segment (start 136.352077 139.5) (end 171.912077 139.5) (width 0.25) (layer "F.Cu") (net 4))
   (segment (start 174.5 107.795923) (end 176.878 107.795923) (width 1.3462) (layer "F.Cu") (net 4))
-  (segment (start 135.845923 139.545923) (end 136.398 139.545923) (width 0.25) (layer "F.Cu") (net 4))
   (segment (start 171.958 120.749923) (end 171.958 113.056) (width 0.25) (layer "F.Cu") (net 4))
-  (segment (start 171.958 139.545923) (end 173.482 138.021923) (width 0.25) (layer "F.Cu") (net 4))
-  (segment (start 173.482 138.021923) (end 173.482 122.273923) (width 0.25) (layer "F.Cu") (net 4))
-  (segment (start 171.912077 139.5) (end 171.958 139.545923) (width 0.25) (layer "F.Cu") (net 4))
   (segment (start 175.514 108.809922) (end 175.452039 108.747961) (width 0.25) (layer "F.Cu") (net 4))
   (segment (start 175.756 109.009923) (end 181.4 114.653923) (width 0.25) (layer "F.Cu") (net 4))
-  (segment (start 136.352077 139.5) (end 136.398 139.545923) (width 0.25) (layer "F.Cu") (net 4))
+  (segment (start 171.958 139.545923) (end 173.482 138.021923) (width 0.25) (layer "F.Cu") (net 4))
   (segment (start 175.514 109.5) (end 175.514 108.809922) (width 0.25) (layer "F.Cu") (net 4))
   (segment (start 171.958 113.056) (end 175.514 109.5) (width 0.25) (layer "F.Cu") (net 4))
+  (segment (start 171.912077 139.5) (end 171.958 139.545923) (width 0.25) (layer "F.Cu") (net 4))
   (segment (start 175.714 109.009923) (end 175.452039 108.747961) (width 0.25) (layer "F.Cu") (net 4))
   (segment (start 175.514 110.4) (end 175.514 109.5) (width 0.25) (layer "F.Cu") (net 4))
   (segment (start 175.756 109.009923) (end 175.714 109.009923) (width 0.25) (layer "F.Cu") (net 4))
-  (segment (start 173.482 122.273923) (end 171.958 120.749923) (width 0.25) (layer "F.Cu") (net 4))
   (segment (start 176.878 107.795923) (end 178.562 106.111923) (width 1.3462) (layer "F.Cu") (net 4))
-  (segment (start 136.352077 139.5) (end 171.912077 139.5) (width 0.25) (layer "F.Cu") (net 4))
+  (segment (start 136.398 139.545923) (end 136.352077 139.5) (width 0.25) (layer "F.Cu") (net 4))
+  (segment (start 173.482 121.3612) (end 171.958 119.8372) (width 0.25) (layer "F.Cu") (net 4))
+  (segment (start 135.845923 139.545923) (end 136.398 139.545923) (width 0.25) (layer "F.Cu") (net 4))
   (segment (start 175.514 113.964923) (end 175.514 110.4) (width 0.25) (layer "F.Cu") (net 4))
   (segment (start 172.958 107.795923) (end 174.5 107.795923) (width 1.3462) (layer "F.Cu") (net 4))
+  (segment (start 132.5 136.2) (end 135.845923 139.545923) (width 0.25) (layer "F.Cu") (net 4))
   (segment (start 160.274 125.067923) (end 159.258 124.051923) (width 0.25) (layer "F.Cu") (net 5))
   (segment (start 169.771923 93.571923) (end 170.8 94.6) (width 1.3462) (layer "F.Cu") (net 5))
@@
   (segment (start 169.926 123.167923) (end 169.926 110.502923) (width 0.25) (layer "F.Cu") (net 6))
   (segment (start 149.446 133.195923) (end 149.446 129.639923) (width 0.25) (layer "F.Cu") (net 7))
+  (segment (start 149.446 130.561924) (end 149.446 130.6068) (width 0.25) (layer "F.Cu") (net 7))
+  (segment (start 154.4 127.4) (end 152.607924 127.4) (width 0.25) (layer "F.Cu") (net 7))
   (segment (start 149.446 128.261923) (end 148.844 127.659923) (width 0.25) (layer "F.Cu") (net 7))
-  (segment (start 150.368001 129.639923) (end 149.446 129.639923) (width 0.25) (layer "F.Cu") (net 7))
-  (segment (start 152.607924 127.4) (end 150.368001 129.639923) (width 0.25) (layer "F.Cu") (net 7))
+  (segment (start 152.607924 127.4) (end 149.446 130.561924) (width 0.25) (layer "F.Cu") (net 7))
   (segment (start 149.446 129.639923) (end 149.446 128.261923) (width 0.25) (layer "F.Cu") (net 7))
-  (segment (start 154.4 127.4) (end 152.607924 127.4) (width 0.25) (layer "F.Cu") (net 7))
   (segment (start 142.24 129.5) (end 142.24 126.813923) (width 0.25) (layer "F.Cu") (net 8))
   (segment (start 142.1 129.5) (end 142.24 129.5) (width 0.25) (layer "F.Cu") (net 8))
@@
   (segment (start 113.2 128.05) (end 111.65 129.6) (width 0.25) (layer "F.Cu") (net 12))
   (segment (start 115.1375 128.05) (end 113.2 128.05) (width 0.25) (layer "F.Cu") (net 12))
-  (segment (start 119.7 131.025) (end 119.7 133.475) (width 0.25) (layer "F.Cu") (net 13))
+  (segment (start 119.7 131.7786) (end 119.7 133.475) (width 0.25) (layer "F.Cu") (net 13))
   (segment (start 120.8625 129.8625) (end 122.475 131.475) (width 0.25) (layer "F.Cu") (net 13))
+  (segment (start 120.8625 130.6161) (end 119.7 131.7786) (width 0.25) (layer "F.Cu") (net 13))
   (segment (start 120.8625 129.35) (end 120.8625 129.8625) (width 0.25) (layer "F.Cu") (net 13))
-  (segment (start 120.8625 129.8625) (end 119.7 131.025) (width 0.25) (layer "F.Cu") (net 13))
+  (segment (start 120.8625 129.8625) (end 120.8625 130.6161) (width 0.25) (layer "F.Cu") (net 13))
   (segment (start 122.475 131.475) (end 123 131.475) (width 0.25) (layer "F.Cu") (net 13))
   (segment (start 179.9 86.132) (end 179.9 84.1) (width 0.25) (layer "F.Cu") (net 14))
@@
   (segment (start 128.4 93.551923) (end 141.117 93.551923) (width 1.3462) (layer "F.Cu") (net 16))
   (segment (start 126.064 93.571923) (end 126.044 93.551923) (width 0.9398) (layer "F.Cu") (net 16))
+  (segment (start 130.048 91.582923) (end 128.4 93.230923) (width 0.25) (layer "F.Cu") (net 16))
+  (segment (start 128.4 93.230923) (end 128.4 93.551923) (width 0.25) (layer "F.Cu") (net 16))
   (segment (start 141.117 93.551923) (end 141.137 93.571923) (width 1.3462) (layer "F.Cu") (net 16))
-  (segment (start 130.048 91.582923) (end 130.048 91.903923) (width 1.3462) (layer "F.Cu") (net 16))
-  (segment (start 130.048 91.903923) (end 128.4 93.551923) (width 1.3462) (layer "F.Cu") (net 16))
   (segment (start 126.044 93.551923) (end 128.4 93.551923) (width 1.3462) (layer "F.Cu") (net 16))
   (segment (start 126.044 91.011923) (end 126.044 96.091923) (width 1.3462) (layer "F.Cu") (net 16))
