File: tank-heating/heater-PCB/heater/heater.kicad_pcb (KiCad board)
At the start: 2 copper layers, 80 x 500 mm, 3 parts, among them J1 Heater connector, J2 Thermistor Connector

Commit message: Add silkscreen, make minor connector position adjustments, and export gerber files
Parts:
- moved J2 34.5 mm to (440.0, 475.5)
- moved J1 6.50 mm to (440.0, 538.5)
Routing:
- net Net-(J2-Pin_2): track 205.3 -> 170.8 mm
- net Net-(J2-Pin_1): track 205.3 -> 170.8 mm
Other:
- board text added: "NO STEP"
- board text added: "Tank Heating V1 - HOT TO GO! Z.Mears 2024-06-10"
