File: Groundside Charging Board Respin/Groundside Charging Board.kicad_sch (KiCad schematic)
At the start: 34 parts, among them M1 60V, M2 60V, M3 60V, M4 40V, U1 TPS43060RTER

Commit message: Add files via upload
Parts:
- removed Iout1: WB_CURRENT_LOAD, symbol TI WEBENCH:Iout
- removed M3: 60V, Package_DIP:DIP-24_W7.62mm, symbol Simulation_SPICE:PMOS
- removed M4: 40V, Package_DFN_QFN:Nordic_AQFN-94-1EP_7x7mm_P0.4mm, symbol Simulation_SPICE:NMOS
- removed R15, R16: CRG1206F10K, symbol TI WEBENCH:Rfbt
- removed Vin1: WB_BATTERY, symbol TI WEBENCH:Vin
- added J1: Conn_01x02, Package_QFP:TQFP-44_10x10mm_P0.8mm, symbol Connector_Generic:Conn_01x02
- added J2: Conn_01x02, symbol Connector_Generic:Conn_01x02
- Rfbb1: value CRG1206F20K -> CRCW040211K0FKED; ALTIUM_VALUE 20k -> 11k; MANUFACTURER NAME TE Connectivity -> Vishay-Dale; MANUFACTURER PART NUMBER CRG1206F20K -> CRCW040211K0FKED; PACKAGEREFERENCE CRG1206F20K -> CRCW040211K0FKED
- Rfbt1: value CRG1206F470K -> CRCW0402261KFKED; ALTIUM_VALUE 470k -> 261k; MANUFACTURER NAME TE Connectivity -> Vishay-Dale; MANUFACTURER PART NUMBER CRG1206F470K -> CRCW0402261KFKED; PACKAGEREFERENCE CRG1206F470K -> CRCW0402261KFKED
Connections:
- net 0: now also J1.2 (Pin_2), J2.2 (Pin_2)
- net at Cin1.1, Cin_2.1, Cvin1.1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: now also J1.1 (Pin_1)
- net at Cout2.1, Cout_1.1, Cout_3.1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: now also J2.1 (Pin_1)
- net EN: no longer names the net of U1.15 (EN)
Other:
- note added: "TI webench link"
- note removed: "Link to IC Datasheet"
- note removed: "To Microcontroller for charging toggling and to M4 Gate"
- moved on the sheet: Cvin1

Commit message: Add files via upload
Parts:
- J1: value Conn_01x02 -> 12V_Input
- J2: value Conn_01x02 -> 30V_Output
Changed lines of the file:
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@@
 			)
 		)
-		(property "Value" "Conn_01x02"
+		(property "Value" "12V_Input"
 			(at 36.83 88.8999 0)
 			(show_name no)
@@
 			)
 		)
-		(property "Value" "Conn_01x02"
+		(property "Value" "30V_Output"
 			(at 439.42 74.9299 0)
 			(show_name no)
